File: christmas_tree_barrier/christmas_tree_barrier.sch (KiCad schematic (older format))
At the start: 15 parts, among them CON1 AVR-ISP-6, IC1 MIC5225-3.3, J1 USB_OTG, J2 JSTPH, J3 JSTPH, Q1 Q_NPN_BEC, U1 ATTINY45-20SU, Y1 8Mhz

Commit message: Fix footprints SOIC-8 was wrong--body was too narrow and pads too short LEDs were unclear--cathode indicator was on top of solder mask area
Also plotted gerbers
Parts:
- U1: footprint lib_fp:SOIC-8_3.9x4.9mm_Pitch1.27mm -> lib_fp:SOIC-8_5.35x5.40mm_Pitch1.27mm
Changed lines of the file:
@@
 Sheet 1 1
 Title "Roomba Christmas Tree Barrier"
-Date "2017-11-30"
-Rev "A"
+Date "2018-01-03"
+Rev "B"
 Comp "Petezah"
 Comment1 "(C) 2017 Peter Dunshee"
@@
 F 0 "U1" H 4650 4100 50  0000 C CNN
 F 1 "ATTINY45-20SU" H 6800 3300 50  0000 C CNN
-F 2 "lib_fp:SOIC-8_3.9x4.9mm_Pitch1.27mm" H 6750 3700 50  0001 C CIN
+F 2 "lib_fp:SOIC-8_5.35x5.40mm_Pitch1.27mm" H 6750 3700 50  0001 C CIN
 F 3 "" H 5800 3700 50  0001 C CNN
 	1    5800 3700
